Commit message: use xacro create a car robot,exist a bug: the car will up in gazebo

File: src/my_robot_description2/urdf/inertial.xacro (robot description, xacro)
@@ -17,3 +17,11 @@
         </inertial>
     </xacro:macro>
+    <xacro:macro name="box_inertial_matrix" params="m l w h">
+        <inertial>
+            <mass value="${m}" />
+            <inertia ixx="${m*(w*w + h*h)/12}" ixy="0" ixz="0"
+                    iyy="${m*(l*l + h*h)/12}" iyz="0"
+                    izz="${m*(l*l + w*w)/12}" />
+        </inertial>
+    </xacro:macro>
 </robot>
