Commit message: add a world demo

File: src/my_robot_description2/urdf/car_base.xacro (robot description, xacro)
@@ -20,5 +20,5 @@
     <xacro:property name="base_height" value="0.28"/>
     <!-- 质量 -->
-    <xacro:property name="base_mass" value="20" />
+    <xacro:property name="base_mass" value="200" />
     <!-- Defining the colors used in this robot -->
     <material name="yellow">
@@ -98,5 +98,5 @@
         </gazebo>
         <xacro:wheel prefix="left" reflect="-1" reflect2="1"/>
-        <xacro:wheel prefix="right" reflect="1" reflect2="1"/>
+        <!-- <xacro:wheel prefix="right" reflect="1" reflect2="1"/> -->
         <!-- <xacro:wheel prefix="left2" reflect="-1" reflect2="-1"/> -->
         <!-- <xacro:wheel prefix="right2" reflect="1" reflect2="-1"/> -->
